Commit message: 15 slope test env

File: tokenhsi/data/assets/carry_box/indented_box.urdf (robot description, URDF)
Before this commit: robot indented_box, 1 links, 0 joints
Links:
- link box: geometry collision mesh filename=indented_box.obj scale=0.41 0.25 0.31; visual mesh filename=indented_box.obj scale=0.41 0.25 0.31

Commit message: CRC experiment

File: tokenhsi/data/assets/carry_box/indented_box.urdf (robot description, URDF)
Before this commit: robot indented_box, 1 links, 0 joints
Links:
- link box: geometry collision mesh filename=indented_box.obj scale=0.4 0.4 0.4; visual mesh filename=indented_box.obj scale=0.4 0.4 0.4
