Commit message: fix for bag with passive joints

File: tokenhsi/data/assets/non_rigid_bag/concrete_bag.urdf (robot description, URDF)
Before this commit: robot concrete_bag_box_chain, 5 links, 4 joints
Links:
- link seg_0: mass 8.0 -> None; geometry collision box size=0.102 0.35 0.12; visual box size=0.102 0.35 0.12
- link seg_1: mass 9.0 -> None; geometry collision box size=0.102 0.35 0.135; visual box size=0.102 0.35 0.135
- link seg_2: mass 10.0 -> None; geometry collision box size=0.102 0.35 0.15; visual box size=0.102 0.35 0.15
- link seg_3: mass 9.0 -> None; geometry collision box size=0.102 0.35 0.135; visual box size=0.102 0.35 0.135
- link seg_4: mass 8.0 -> None; geometry collision box size=0.102 0.35 0.12; visual box size=0.102 0.35 0.12
Joints:
- joint j_0_1: limit lower=-0.785 upper=0.785 effort=500 velocity=2.0 -> lower=-0.133 upper=0.133 effort=500 velocity=2.0; origin xyz=0.061 0 0 rpy=0 0 0 -> xyz=0.122 0 0 rpy=0 0 0; type fixed -> revolute
- joint j_1_2: limit lower=-0.785 upper=0.785 effort=500 velocity=2.0 -> lower=-0.133 upper=0.133 effort=500 velocity=2.0; origin xyz=0.061 0 0 rpy=0 0 0 -> xyz=0.122 0 0 rpy=0 0 0; type fixed -> revolute
- joint j_2_3: limit lower=-0.785 upper=0.785 effort=500 velocity=2.0 -> lower=-0.133 upper=0.133 effort=500 velocity=2.0; origin xyz=0.061 0 0 rpy=0 0 0 -> xyz=0.122 0 0 rpy=0 0 0; type fixed -> revolute
- joint j_3_4: limit lower=-0.785 upper=0.785 effort=500 velocity=2.0 -> lower=-0.133 upper=0.133 effort=500 velocity=2.0; origin xyz=0.061 0 0 rpy=0 0 0 -> xyz=0.122 0 0 rpy=0 0 0; type fixed -> revolute

Commit message: bag training setup

File: tokenhsi/data/assets/non_rigid_bag/concrete_bag.urdf (robot description, URDF)
Before this commit: robot concrete_bag_box_chain, 5 links, 4 joints
Links:
- link seg_0: geometry collision box size=0.35 0.102 0.12; visual box size=0.35 0.102 0.12
- link seg_1: geometry collision box size=0.35 0.102 0.135; visual box size=0.35 0.102 0.135
- link seg_2: geometry collision box size=0.35 0.102 0.15; visual box size=0.35 0.102 0.15
- link seg_3: geometry collision box size=0.35 0.102 0.135; visual box size=0.35 0.102 0.135
- link seg_4: geometry collision box size=0.35 0.102 0.12; visual box size=0.35 0.102 0.12
Joints:
- removed joint j_0_1
- removed joint j_1_2
- added joint j_1_0: type revolute, parent seg_1, child seg_0, origin xyz=0 -0.122 0 rpy=0 0 0, axis 1 0 0, limit lower=-0.133 upper=0.133 effort=500 velocity=2.0
- added joint j_2_1: type revolute, parent seg_2, child seg_1, origin xyz=0 -0.122 0 rpy=0 0 0, axis 1 0 0, limit lower=-0.133 upper=0.133 effort=500 velocity=2.0
- joint j_2_3: axis 0 1 0 -> 1 0 0; origin xyz=0.122 0 0 rpy=0 0 0 -> xyz=0 0.122 0 rpy=0 0 0
- joint j_3_4: axis 0 1 0 -> 1 0 0; origin xyz=0.122 0 0 rpy=0 0 0 -> xyz=0 0.122 0 rpy=0 0 0
