Commit message: flat experiments

File: tokenhsi/data/assets/non_rigid_bag/stone_bag_l.urdf (robot description, URDF)
Before this commit: robot stone_bag_box_chain, 5 links, 4 joints
Links:
- link seg_0: geometry collision box size=0.35 0.102 0.12; visual box size=0.35 0.102 0.12
- link seg_1: geometry collision box size=0.35 0.102 0.135; visual box size=0.35 0.102 0.135
- link seg_2: geometry collision box size=0.35 0.102 0.15; visual box size=0.35 0.102 0.15
- link seg_3: geometry collision box size=0.35 0.102 0.135; visual box size=0.35 0.102 0.135
- link seg_4: geometry collision box size=0.35 0.102 0.12; visual box size=0.35 0.102 0.12
Joints:
- joint j_1_0: origin xyz=0 -0.1077 0 rpy=0 0 0 -> xyz=0 -0.122 0 rpy=0 0 0
- joint j_2_1: origin xyz=0 -0.1077 0 rpy=0 0 0 -> xyz=0 -0.122 0 rpy=0 0 0
- joint j_2_3: origin xyz=0 0.1077 0 rpy=0 0 0 -> xyz=0 0.122 0 rpy=0 0 0
- joint j_3_4: origin xyz=0 0.1077 0 rpy=0 0 0 -> xyz=0 0.122 0 rpy=0 0 0
